File: StereoAmigaAudioDigitizer.kicad_pcb (KiCad board)
At the start: 2 copper layers, 54.4 x 44.7 mm, 22 parts, among them J1 RIGHT, J2 LEFT, J3 DB25_Male, U1 MCP6002, U2 DG419LDJ, U3 ADC0820CCN+

Commit message: Add files via upload
Modified PCB
Parts:
- J1: footprint w_conn_av:rca_red -> w_conn_av:rca_white
- J3: footprint Connector_Dsub:DSUB-25_Male_Horizontal_P2.77x2.84mm_EdgePinOffset4.94mm_Housed_MountingHolesOffset7.48mm -> Connector_Dsub:DSUB-25_Male_Horizontal_P2.77x2.84mm_EdgePinOffset7.70mm_Housed_MountingHolesOffset9.12mm
- moved J1 0.45 mm to (140.5, 86.2)
- moved J2 0.40 mm to (125.0, 86.2)
- renumbered VOLUME to RV1
Other:
- board size 54.4 x 44.7 mm -> 54.4 x 45.1 mm
- board text added: "AMIGA STEREO DIGITIZER V1.2"
- board text added: "GAIN"
- board text removed: "AMIGA STEREO DIGITIZER V1.1"

Commit message: Add files via upload
Parts:
- removed C8: 10uF, Capacitor_THT:CP_Radial_D4.0mm_P1.50mm
- removed G***: LOGO, Symbol:openhardware
- removed the R1 at (100.3, 59.9)
- removed the R2 at (98.0, 70.6)
- added LOGO1: OSHW-Logo_5.7x6mm_Copper, Symbol:OSHW-Logo_5.7x6mm_Copper, B.Cu at (136.2, 75.9)
- added LOGO2: LOGO, Symbol:pcm, B.Cu at (121.0, 63.8)
- added LOGO3: LOGO, Symbol:RetronicDesign, B.Cu at (122.9, 49.7)
- RV1: value 10K exp -> A10K; footprint Potentiometer_THT:Potentiometer_Alps_RK09L_Double_Horizontal -> Potentiometer_THT:Potentiometer_Alps_RK09K_Single_Horizontal
- U2: value DG419LDJ -> DG419DJ
- U3: value ADC0820CCN+ -> ADC0820CCN
- moved C4 21.7 mm to (99.2, 62.2)
- moved C5 18.6 mm to (117.1, 77.8), turned to 0 degrees
- moved R3 18.1 mm to (116.1, 71.6), turned to 180 degrees
- moved U2 15.4 mm to (114.5, 81.1), turned to 0 degrees
- moved U1 11.0 mm to (102.5, 67.5)
- moved R4 10.9 mm to (106.7, 71.6), turned to 180 degrees
- moved C2 5.75 mm to (142.4, 72.3)
- moved R2 5.66 mm to (132.5, 76.0)
- moved J1 5.18 mm to (130.2, 86.1)
- moved C3 5.16 mm to (106.6, 75.2)
- moved RV1 3.42 mm to (102.8, 86.7)
- moved C6 3.30 mm to (114.3, 64.9)
- moved U3 3.30 mm to (117.9, 67.5)
- moved C1 2.88 mm to (130.2, 72.4)
- moved C7 2.35 mm to (145.8, 62.7)
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- renumbered C2 to C1, C1 to C2, C7 to C3, C3 to C4, C4 to C5, C5 to C6, C6 to C7, J2 to J1, J1 to J2, R6 to R1, R5 to R2
Connections:
- C3 pad 1: Net-(R3-Pad2) -> Net-(C3-Pad1)
- R1 pad 1: Net-(R6-Pad1) -> Net-(R1-Pad1)
- R2 pad 1: Net-(R5-Pad1) -> Net-(R2-Pad1)
- R3 pad 2: Net-(R3-Pad2) -> Net-(C3-Pad1)
- R4 pad 1: Net-(R3-Pad2) -> Net-(C3-Pad1)
- RV1 pad 1: Net-(R6-Pad1) -> Net-(RV1-Pad1)
- U1 pad 2: Net-(R3-Pad2) -> Net-(U1-Pad2)
- U1 pad 3: Net-(R6-Pad1) -> Net-(RV1-Pad1)
- U1 pad 5: Net-(R5-Pad1) -> Net-(U1-Pad2)
- U1 pad 6: Net-(R1-Pad2) -> Net-(C3-Pad1)
- U1 pad 7: Net-(RV1-Pad5) -> Net-(U1-Pad2)
- U2 pad 1: Net-(U3-Pad1) -> Net-(RV1-Pad1)
- U2 pad 2: Net-(RV1-Pad2) -> Net-(R1-Pad1)
- U2 pad 8: Net-(RV1-Pad5) -> Net-(R2-Pad1)
- U3 pad 1: Net-(U3-Pad1) -> unconnected-(U3-Pad1)
Routing:
- net //SELECT: track 6.95 -> 49.2 mm
- net Net-(R5-Pad1): track 41.5 -> 0.00 mm
- net Net-(RV1-Pad5): track 37.3 -> 0.00 mm
- net Net-(RV1-Pad1): track 0.00 -> 33.4 mm
- net Net-(R6-Pad1): track 33.2 -> 0.00 mm
- net Net-(C3-Pad1): track 0.00 -> 26.4 mm
- net //STROBE: track 15.3 -> 38.8 mm
- net Net-(R1-Pad2): track 18.5 -> 0.00 mm
- net Net-(R3-Pad2): track 15.5 -> 0.00 mm
- net Net-(U3-Pad1): track 15.4 -> 0.00 mm
- net Net-(U1-Pad2): track 0.00 -> 14.6 mm
- net Net-(RV1-Pad2): track 36.6 -> 22.8 mm
- net Net-(R2-Pad1): track 0.00 -> 12.6 mm
- net Net-(R1-Pad1): track 0.00 -> 12.5 mm
- net /D1: track 17.8 -> 26.0 mm
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Other:
- board text added: "8-bit"
- board text added: "AMIGA STEREO DIGITIZER V1.3"
- board text added: "GND"
- board text added: "INPUT GAIN"
- board text added: "VGND=+2.5V"
- board text added: "WWW.RETRONICDESIGN.COM"
- board text removed: "AMIGA STEREO DIGITIZER V1.2"
- board text removed: "GAIN"
- board text removed: "RETRONICDESIGN.COM OPEN HARDWARE LICENSE"
