File: StereoAmigaAudioDigitizer.kicad_pcb (KiCad board)
At the start: 2 copper layers, 54.4 x 45.1 mm, 21 parts, among them J1 LEFT, J2 RIGHT, J3 DB25_Male, U1 MCP6002, U2 DG419DJ, U3 ADC0820CCN

Commit message: Add files via upload
1.3a
Parts:
- moved C5 10.5 mm to (117.0, 88.3)
- moved U2 4.10 mm to (114.5, 77.0)
- moved R4 0.43 mm to (106.4, 71.2)
- moved R3 0.35 mm to (116.1, 71.2)
Connections:
- U3 pad 1: unconnected-(U3-Pad1) -> Net-(RV1-Pad2)
Routing:
- net Net-(RV1-Pad2): track 22.8 -> 53.3 mm
- net //STROBE: track 38.8 -> 30.3 mm
- net Net-(RV1-Pad1): track 33.4 -> 29.8 mm
- net +5V: track 113.8 -> 116.9 mm
- net //SELECT: track 49.2 -> 46.7 mm
- net Net-(R1-Pad1): track 12.5 -> 11.0 mm
- net Net-(R2-Pad1): track 12.6 -> 11.0 mm
Other:
- board text added: "AMIGA STEREO DIGITIZER V1.3a"
- board text added: "stereo"
- board text removed: "AMIGA STEREO DIGITIZER V1.3"
