File: StereoAmigaAudioDigitizer.kicad_sch (KiCad schematic)
At the start: 21 parts, among them J1 RIGHT, J2 LEFT, J3 DB25_Male, U1 MCP6002, U2 DG419DJ, U3 ADC0820CCN+

Commit message: Add files via upload
Modified PCB
Other:
- moved on the sheet: C4, C5, U2B

Commit message: Add files via upload
Parts:
- removed C8: 10uF, Capacitor_THT:CP_Radial_D5.0mm_P2.50mm, symbol Device:C_Polarized_US
- removed R1, R2: 1K, Resistor_THT:R_Axial_DIN0204_L3.6mm_D1.6mm_P2.54mm_Vertical, symbol Device:R
- removed RV1: 10K exp, Potentiometer_THT:Potentiometer_Alps_RK09L_Double_Horizontal, symbol Device:R_Potentiometer_Dual_Separate
- removed U1: MCP6002, Package_DIP:DIP-8_W7.62mm, symbol Amplifier_Operational:MCP6002-xMC
- added RV1: A10K, Potentiometer_THT:Potentiometer_Alps_RK09K_Single_Vertical, symbol Device:R_Potentiometer_US
- added U1: MCP6002, Package_DIP:DIP-8_W7.62mm, symbol Amplifier_Operational:MCP6002-xMS
- C1: renamed from C2; footprint Capacitor_THT:CP_Radial_D5.0mm_P2.50mm -> Capacitor_THT:CP_Radial_D4.0mm_P1.50mm
- C2: renamed from C1; footprint Capacitor_THT:CP_Radial_D5.0mm_P2.50mm -> Capacitor_THT:CP_Radial_D4.0mm_P1.50mm
- C3: renamed from C7; footprint Capacitor_THT:CP_Radial_D5.0mm_P2.50mm -> Capacitor_THT:CP_Radial_D4.0mm_P1.50mm
- C7: renamed from C6; footprint Capacitor_THT:CP_Radial_D5.0mm_P2.50mm -> Capacitor_THT:CP_Radial_D4.0mm_P1.50mm
- J3: footprint Connector_Dsub:DSUB-25_Male_Horizontal_P2.77x2.84mm_EdgePinOffset4.94mm_Housed_MountingHolesOffset7.48mm -> Connector_Dsub:DSUB-25_Male_Horizontal_P2.77x2.84mm_EdgePinOffset7.70mm_Housed_MountingHolesOffset9.12mm
- R3, R4: footprint Resistor_THT:R_Axial_DIN0204_L3.6mm_D1.6mm_P2.54mm_Vertical -> Resistor_THT:R_Axial_DIN0204_L3.6mm_D1.6mm_P7.62mm_Horizontal
- U3: value ADC0820CCN+ -> ADC0820CCN
- renumbered C3 to C4, C4 to C5, C5 to C6, J2 to J1, J1 to J2, R6 to R1, R5 to R2
Connections:
- net +5V: now also U1.8 (V+)
- net GND: now also U1.4 (V-)
- net at U2.1: now also RV1.1, U1.3 (+); no longer U3.1 (Vin)
- net at C3.1, R3.2, R4.1: now also U1.6 (-)
- net at U2.2: now also R1.1
- net at U2.8: now also R2.1
- new net: RV1.2, RV1.3, U1.1
- new net: U1.2 (-), U1.5 (+), U1.7
Other:
- note added: "VIRTUAL GROUND (2.5V)"
- note removed: "DC OFFSET"
- moved on the sheet: C1, C2, C3, C4, C5, C6, C7, J1, J2, J3, R1, R2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
