File: StereoAmigaAudioDigitizer.kicad_sch (KiCad schematic)
At the start: 18 parts, among them J1 LEFT, J2 RIGHT, J3 DB25_Male, U1 MCP6002, U2 DG419DJ, U3 ADC0820CCN

Commit message: Add files via upload
1.3a
Parts:
- U2: value DG419DJ -> ADG419BNZ
Connections:
- net GND: no longer U2.3 (GND)
Other:
- moved on the sheet: C5, C6
